Commit message: Ampliación de límites de giro en URDF (Joints 8, 9, 12) y corrección de rutas de paquetes

File: yaren_description/urdf/yaren_description.urdf (robot description, URDF)
Before this commit: robot yaren_description, 15 links, 14 joints
Joints:
- joint joint_1: limit lower=-0.7853 upper=0.7853 effort=300 velocity=3 -> lower=-3.1416 upper=3.1416 effort=300 velocity=3
- joint joint_10: limit lower=0 upper=1.0472 effort=300 velocity=3 -> lower=-3.1416 upper=3.1416 effort=300 velocity=3
- joint joint_11: limit lower=-0.7853 upper=0.7853 effort=300 velocity=3 -> lower=-3.1416 upper=3.1416 effort=300 velocity=3
- joint joint_12: limit lower=0.1745 upper=1.5708 effort=300 velocity=3 -> lower=-3.1416 upper=3.1416 effort=300 velocity=3
- joint joint_2: limit lower=-0.5235 upper=0.5235 effort=300 velocity=3 -> lower=-3.1416 upper=3.1416 effort=300 velocity=3
- joint joint_3: limit lower=-0.5235 upper=0.5235 effort=300 velocity=3 -> lower=-3.1416 upper=3.1416 effort=300 velocity=3
- joint joint_4: limit lower=-0.2617 upper=0.7853 effort=300 velocity=3 -> lower=-3.1416 upper=3.1416 effort=300 velocity=3
- joint joint_5: limit lower=-0.7853 upper=1.5708 effort=300 velocity=3 -> lower=-3.1416 upper=3.1416 effort=300 velocity=3
- joint joint_6: limit lower=0 upper=1.0472 effort=300 velocity=3 -> lower=-3.1416 upper=3.1416 effort=300 velocity=3
- joint joint_7: limit lower=-0.7853 upper=0.7853 effort=300 velocity=3 -> lower=-3.1416 upper=3.1416 effort=300 velocity=3
- joint joint_8: limit lower=0.1745 upper=1.5708 effort=300 velocity=3 -> lower=-3.1416 upper=3.1416 effort=300 velocity=3
- joint joint_9: limit lower=-0.7853 upper=1.5708 effort=300 velocity=3 -> lower=-3.1416 upper=3.1416 effort=300 velocity=3

Commit message: Actualiza URDF, lógica de expresiones faciales, configs de U2D2 y añade script go_base

File: yaren_description/urdf/yaren_description.urdf (robot description, URDF)
Before this commit: robot yaren_description, 15 links, 14 joints
Links:
- removed link camera_link
- link base_link: mass 1.36786443462294 -> 1.3678
- link link_1: mass 0.2613 -> None; geometry visual mesh filename=package://yaren_description/meshes/Link_1.STL
- link link_10: mass 0.0569176449626118 -> None; geometry visual mesh filename=package://yaren_description/meshes/Link_10.STL
- link link_11: mass 0.112981340262659 -> None; geometry visual mesh filename=package://yaren_description/meshes/Link_11.STL
- link link_12: mass 0.040449 -> None; geometry visual mesh filename=package://yaren_description/meshes/Link_12.STL
- link link_2: mass 0.752173682094854 -> None; geometry visual mesh filename=package://yaren_description/meshes/Link_2.STL
- link link_3: mass 0.0569176449626117 -> None; geometry visual mesh filename=package://yaren_description/meshes/Link_3.STL
- link link_4: mass 0.654995275916393 -> None; geometry visual mesh filename=package://yaren_description/meshes/Link_4.STL
- link link_5: mass 0.0584361592248743 -> None; geometry visual mesh filename=package://yaren_description/meshes/Link_5.STL
- link link_6: mass 0.056918 -> None; geometry visual mesh filename=package://yaren_description/meshes/Link_6.STL
- link link_7: mass 0.11298 -> None; geometry visual mesh filename=package://yaren_description/meshes/Link_7.STL
- link link_8: mass 0.0489075786054985 -> None; geometry visual mesh filename=package://yaren_description/meshes/Link_8.STL
- link link_9: mass 0.0584361879389782 -> None; geometry visual mesh filename=package://yaren_description/meshes/Link_9.STL
Joints:
- removed joint camera_joint
- joint joint_1: limit lower=-3.1416 upper=3.1416 effort=300 velocity=3 -> lower=-10.0 upper=10.0 effort=300 velocity=3; origin xyz=0.0 0.0 0.020523 rpy=1.5708 0 1.5708 -> xyz=0.0 0.0 0.020523 rpy=1.5708 0 1.6008
- joint joint_10: limit lower=-3.1416 upper=3.1416 effort=300 velocity=3 -> lower=-10.0 upper=10.0 effort=300 velocity=3; origin xyz=-0.031745769115688 -0.0195 0 rpy=0 0 -1.5707963267949 -> xyz=-0.031745 -0.0195 0 rpy=0 0 -1.6108
- joint joint_11: limit lower=-3.1416 upper=3.1416 effort=300 velocity=3 -> lower=-10.0 upper=10.0 effort=300 velocity=3; origin xyz=0.0190000001524479 -0.0240000007161399 -0.000529483238776968 rpy=-1.5707963267949 0 0 -> xyz=0.019 -0.024 -0.0005 rpy=-1.4808 0 0
- joint joint_12: limit lower=-3.1416 upper=3.1416 effort=300 velocity=3 -> lower=-10.0 upper=10.0 effort=300 velocity=3; origin xyz=0.09125 0 0 rpy=1.5707963267949 0 -2.91667493011268 -> xyz=0.09125 0 0 rpy=1.5708 0 -2.5867
- joint joint_2: limit lower=-3.1416 upper=3.1416 effort=300 velocity=3 -> lower=-10.0 upper=10.0 effort=300 velocity=3
- joint joint_3: limit lower=-3.1416 upper=3.1416 effort=300 velocity=3 -> lower=-10.0 upper=10.0 effort=300 velocity=3; origin xyz=0 0.1145 -0.012 rpy=-1.5708 0 0 -> xyz=0 0.1145 -0.012 rpy=-1.5908 0 0
- joint joint_4: limit lower=-3.1416 upper=3.1416 effort=300 velocity=3 -> lower=-10.0 upper=10.0 effort=300 velocity=3; origin xyz=0 -0.024 0.02 rpy=1.5708 0 1.5708 -> xyz=0 -0.024 0.02 rpy=1.5708 0 1.5508
- joint joint_5: limit lower=-3.1416 upper=3.1416 effort=300 velocity=3 -> lower=-10.0 upper=10.0 effort=300 velocity=3; origin xyz=0.10575 0.09925 0 rpy=3.1416 0 3.1416 -> xyz=0.10575 0.09925 0 rpy=3.1616 0 3.1416
- joint joint_6: limit lower=-3.1416 upper=3.1416 effort=300 velocity=3 -> lower=-10.0 upper=10.0 effort=300 velocity=3
- joint joint_7: limit lower=-3.1416 upper=3.1416 effort=300 velocity=3 -> lower=-10.0 upper=10.0 effort=300 velocity=3; origin xyz=0.019 -0.024 0.00047052 rpy=1.5708 0 0 -> xyz=0.019 -0.024 0.00047 rpy=1.5808 0 0
- joint joint_8: limit lower=-3.1416 upper=3.1416 effort=300 velocity=3 -> lower=-10.0 upper=10.0 effort=300 velocity=3; origin xyz=0.09125 0 0 rpy=1.5708 0 -2.9337 -> xyz=0.09125 0 0 rpy=1.5708 0 -2.5937
- joint joint_9: limit lower=-3.1416 upper=3.1416 effort=300 velocity=3 -> lower=-10.0 upper=10.0 effort=300 velocity=3; origin xyz=-0.105754230884312 0.0992500000000003 0 rpy=0 0 0 -> xyz=-0.10575 0.09925 0 rpy=-0.14 0 0

Commit message: Añadí varios carpetas para Yaren en ros2 humble

File: yaren_description/urdf/yaren_description.urdf (robot description, URDF)
Before this commit: robot yaren_description, 14 links, 13 joints
Joints:
- joint joint_9: axis 1 0 0 -> -1 0 0

File: yaren_description/urdf/yaren_description_sim.xacro.urdf (robot description, URDF)
Before this commit: robot yaren_description_sim, 15 links, 14 joints
Joints:
- joint joint_1: limit lower=-0.7853 upper=0.7853 effort=300 velocity=3 -> lower=-3.1416 upper=3.1416 effort=300 velocity=3
- joint joint_10: limit lower=0 upper=1.0472 effort=300 velocity=3 -> lower=-3.1416 upper=3.1416 effort=300 velocity=3
- joint joint_11: limit lower=-0.7853 upper=0.7853 effort=300 velocity=3 -> lower=-3.1416 upper=3.1416 effort=300 velocity=3
- joint joint_12: limit lower=0.1745 upper=1.5708 effort=300 velocity=3 -> lower=-3.1416 upper=3.1416 effort=300 velocity=3
- joint joint_2: limit lower=-0.5235 upper=0.5235 effort=300 velocity=3 -> lower=0.0 upper=0.0 effort=300 velocity=0
- joint joint_3: limit lower=-0.5235 upper=0.5235 effort=300 velocity=3 -> lower=-3.1416 upper=3.1416 effort=300 velocity=3
- joint joint_4: limit lower=-0.2617 upper=0.7853 effort=300 velocity=3 -> lower=-3.1416 upper=3.1416 effort=300 velocity=3
- joint joint_5: limit lower=-0.7853 upper=1.5708 effort=300 velocity=3 -> lower=-3.1416 upper=3.1416 effort=300 velocity=3
- joint joint_6: limit lower=0.000 upper=1.0472 effort=300 velocity=3 -> lower=-3.1416 upper=3.1416 effort=300 velocity=3
- joint joint_7: limit lower=-0.7853 upper=0.7853 effort=300 velocity=3 -> lower=-3.1416 upper=3.1416 effort=300 velocity=3
- joint joint_8: limit lower=0.1745 upper=1.5708 effort=300 velocity=3 -> lower=-3.1416 upper=3.1416 effort=300 velocity=3
- joint joint_9: axis 1 0 0 -> -1 0 0; limit lower=-0.7853 upper=1.5708 effort=300 velocity=3 -> lower=-3.1416 upper=3.1416 effort=300 velocity=3
